Commit message: Modify robot models and others

File: model/franka_panda.urdf (robot description, URDF)
Before this commit: robot panda, 11 links, 10 joints
Joints:
- joint panda_joint1: limit lower=-2.8973 upper=2.8973 effort=87 velocity=2.1750 -> lower=-2.8973 upper=2.8973 effort=87 velocity=10
- joint panda_joint2: limit lower=-1.7628 upper=1.7628 effort=87 velocity=2.1750 -> lower=-1.7628 upper=1.7628 effort=87 velocity=10
- joint panda_joint3: limit lower=-2.8973 upper=2.8973 effort=87 velocity=2.1750 -> lower=-2.8973 upper=2.8973 effort=87 velocity=10
- joint panda_joint4: limit lower=-3.0718 upper=-0.0698 effort=87 velocity=2.1750 -> lower=-3.002 upper=0 effort=87 velocity=10
- joint panda_joint5: limit lower=-2.8973 upper=2.8973 effort=12 velocity=2.6100 -> lower=-2.8973 upper=2.8973 effort=12 velocity=10
- joint panda_joint6: limit lower=-0.0175 upper=3.7525 effort=12 velocity=2.6100 -> lower=-1.588 upper=2.1817 effort=12 velocity=10
- joint panda_joint7: limit lower=-3.14 upper=3.14 effort=12 velocity=2.6100 -> lower=-3.14 upper=3.14 effort=12 velocity=10; origin xyz=0.088 0 0 rpy=1.57079632679 0.84 0 -> xyz=0.088 0 0 rpy=1.57079632679 0 0

File: model/franka_panda_rviz.urdf (robot description, URDF)
Before this commit: robot panda, 11 links, 10 joints
Joints:
- joint panda_joint4: limit lower=-3.0718 upper=-0.0698 effort=87 velocity=2.1750 -> lower=-3.002 upper=0 effort=87 velocity=2.1750
- joint panda_joint6: limit lower=-0.0175 upper=3.7525 effort=12 velocity=2.6100 -> lower=-1.588 upper=2.1817 effort=12 velocity=2.6100; origin xyz=0 0 0 rpy=1.57079632679 0 0 -> xyz=0 0 0 rpy=1.57079632679 -1.57079632679 0
- joint panda_joint7: origin xyz=0.088 0 0 rpy=1.57079632679 0.84 0 -> xyz=0.088 0 0 rpy=1.57079632679 0 0

Commit message: Modify the models

File: model/franka_panda.urdf (robot description, URDF)
Before this commit: robot panda, 11 links, 10 joints
Links:
- added link panda_link8
- link panda_hand: mass 0.68 -> 0.73
- link panda_leftfinger: mass 0.01 -> 0.015
- link panda_link0: mass 3.06 -> 0.629769
- link panda_rightfinger: mass 0.01 -> 0.015
Joints:
- added joint panda_joint8: type fixed, parent panda_link7, child panda_link8, origin xyz=0 0 0.107 rpy=0 0 0, axis 0 0 0
- joint panda_finger_joint1: limit lower=0.0 upper=0.04 effort=20 velocity=0.2 -> lower=0 upper=0.04 effort=20 velocity=0.2; origin xyz=0 0 0.0584 rpy=0 0 0 -> xyz=0 0 0.17 rpy=0 0 -0.7833999
- joint panda_finger_joint2: limit lower=0.0 upper=0.04 effort=20 velocity=0.2 -> lower=0 upper=0.04 effort=20 velocity=0.2; origin xyz=0 0 0.0584 rpy=0 0 0 -> xyz=0 0 0.17 rpy=0 0 -0.7833999
- joint panda_hand_joint: origin xyz=0 0 0.107 rpy=0 0 -1.57 -> xyz=0 0 0 rpy=0 0 -0.785398163397; parent panda_link7 -> panda_link8
- joint panda_joint1: limit lower=-2.8973 upper=2.8973 effort=87 velocity=10 -> lower=-2.9 upper=2.9 effort=87 velocity=2.1750; origin xyz=0 0 0.333 rpy=0 0 0 -> xyz=0 0 0.33 rpy=0 0 0
- joint panda_joint2: limit lower=-1.7628 upper=1.7628 effort=87 velocity=10 -> lower=-1.8 upper=1.8 effort=87 velocity=2.1750; origin xyz=0 0 0 rpy=-1.57079632679 0 0 -> xyz=0 0 0 rpy=-1.5707 0 0
- joint panda_joint3: limit lower=-2.8973 upper=2.8973 effort=87 velocity=10 -> lower=-2.9 upper=2.9 effort=87 velocity=2.1750; origin xyz=0 -0.316 0 rpy=1.57079632679 0 0 -> xyz=0 -0.32 0 rpy=1.5707 0 0
- joint panda_joint4: limit lower=-3.002 upper=0 effort=87 velocity=10 -> lower=-3.1 upper=-0.4 effort=87 velocity=2.1750; origin xyz=0.0825 0 0 rpy=1.57079632679 0 0 -> xyz=0.083 0 0 rpy=1.5707 0 0
- joint panda_joint5: limit lower=-2.8973 upper=2.8973 effort=12 velocity=10 -> lower=-2.9 upper=2.9 effort=12 velocity=2.6100; origin xyz=-0.0825 0.384 0 rpy=-1.57079632679 0 0 -> xyz=-0.083 0.38 0 rpy=-1.5707 0 0
- joint panda_joint6: limit lower=-1.588 upper=2.1817 effort=12 velocity=10 -> lower=-1.7 upper=2.1 effort=12 velocity=2.6100; origin xyz=0 0 0 rpy=1.57079632679 0 0 -> xyz=0 0 0 rpy=1.5707963 0 1.5707963
- joint panda_joint7: limit lower=-3.14 upper=3.14 effort=12 velocity=10 -> lower=-2.9 upper=2.9 effort=12 velocity=2.6100; origin xyz=0.088 0 0 rpy=1.57079632679 0 0 -> xyz=0.088 0 0 rpy=1.5707963 0 0.7873965
